File: kicad/nucleo_f411re_mecanum/nucleo_f411re_mecanum.kicad_sch (KiCad schematic)
At the start: 7 parts, among them U1 NUCLEO64-F411RE

Commit message: better schematic
Parts:
- added U2: ESP32-CAM, ESP32-CAM:ESP32-CAM, symbol ESP32-CAM:ESP32-CAM
Connections:
- net +5V: now also U2.P$9 (5V)
- net GND: now also U2.P$10 (GND@3)
- net USART6_RX renamed ESP32-CAM_TX
- net ESP32-CAM_TX: now also U2.P$12 (GPIO13)
- net USART6_TX renamed ESP32-CAM_RX
- net ESP32-CAM_RX: now also U2.P$11 (GPIO12)
Other:
- company: (none) -> ITIS E.MATTEI URBINO
- title: (none) -> Rover mecanum
- moved on the sheet: BACK, BL, BR, FL, FR, FRONT, U1
